File: NK2_2026_LineSensor_v2/line/line.kicad_sch (KiCad schematic)
At the start: 90 parts, among them J1 Conn_01x05_Socket, J2 Conn_01x07_Socket, J3 Conn_01x07_Socket, J4 Conn_01x07_Socket, J5 Conn_01x02_Socket, J6 Conn_01x02_Socket, J7 USB_C_Receptacle_USB2.0_16P, Q1 Q_Photo_NPN, Q10 Q_Photo_NPN, Q11 Q_Photo_NPN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

Commit message: コネクタの位置を変えた
Parts:
- removed SW1: SW_SPDT, tgl:slide switch, symbol Switch:SW_SPDT
- added C35: 10, Capacitor_SMD:C_0603_1608Metric, symbol Device:C
- added C36: 22, Capacitor_SMD:C_1206_3216Metric, symbol Device:C
- added C9: 100n, Capacitor_SMD:C_0402_1005Metric, symbol Device:C
- added CR1, CR2: SS14, SS14:CR_SMA_403AE_OSI, symbol SS14:SS14
- added J10, J11, J8, J9: Conn_01x04_Socket, Connector_JST:JST_XH_B4B-XH-A_1x04_P2.50mm_Vertical, symbol Connector:Conn_01x04_Socket
- added J12: Conn_01x02_Socket, Connector_JST:JST_XH_B2B-XH-A_1x02_P2.50mm_Vertical, symbol Connector:Conn_01x02_Socket
- added Q13, Q14: DMG2301L-7, DMG2301L-7:SOT96P240X115-3N, symbol DMG2301L-7:DMG2301L-7
- added R42, R43: 10k, Resistor_SMD:R_0603_1608Metric, symbol Device:R
- added SW1: OS102011MA1QN1, SK-12D11VG3:OS102011MA1QN1_CNK, symbol SK-12D11VG3:OS102011MA1QN1
- added U7: AZ1117CH-3.3TRG1, AZ1117CH-3.3TRG1:SOT-223_DIO, symbol AZ1117CH-3.3TRG1:AZ1117CH-3.3TRG1
- C26: value 0.1u -> 100n; footprint (none) -> Capacitor_SMD:C_0402_1005Metric; LCSC (none) -> C1525
- D17: footprint (none) -> LED_SMD:LED_0603_1608Metric; LCSC (none) -> C2286
- J1: footprint (none) -> Connector_JST:JST_XH_S5B-XH-A-1_1x05_P2.50mm_Horizontal
- J2, J3, J4: footprint (none) -> Connector_PinSocket_2.54mm:PinSocket_1x07_P2.54mm_Vertical
- J5, J6: footprint (none) -> Connector_JST:JST_XH_B2B-XH-A_1x02_P2.50mm_Vertical
- J7: LCSC (none) -> C393939
- R1, R18, R20, R22, R24, R26, R28, R31, R33, R35, R37, R39, R4, R40, R41: footprint (none) -> Resistor_SMD:R_0603_1608Metric
- R10, R11, R12, R13, R14, R15, R16, R5, R6, R7, R8, R9: LCSC C17957 -> (none)
- R17, R19, R2, R21, R23, R27, R29, R3, R30, R32, R34, R36, R38: LCSC C15401 -> (none)
- R25: value 10k -> 100k; LCSC C15401 -> (none)
- U1: LCSC (none) -> C47361296
- U4: LCSC (none) -> C99652
- Y1: LCSC (none) -> C32180
Connections:
- net +3.3V: now also C9.1, CR2.1, J10.4 (Pin_4), J11.4 (Pin_4), J8.4 (Pin_4), J9.4 (Pin_4), Q14.2 (S), R43.2; no longer J1.1 (Pin_1), J5.2 (Pin_2), R29.2
- net 5v_1: now also C35.1, U7.3 (INPUT)
- net BOOT0: now also SW1.2
- net GND: now also R29.2, C35.2, C36.2, C9.2, J10.1 (Pin_1), J11.1 (Pin_1), J8.1 (Pin_1), J9.1 (Pin_1), R42.1, U7.1 (ADJ/GND), U7.4 (EPAD)
- net M1_en_1: now also J8.2 (Pin_2)
- net M1_en_2: now also J8.3 (Pin_3)
- net M2_en_1: now also J9.2 (Pin_2)
- net M2_en_2: now also J9.3 (Pin_3)
- net M3_en_1: now also J10.2 (Pin_2)
- net M3_en_2: now also J10.3 (Pin_3)
- net M4_en_1: now also J11.2 (Pin_2)
- net M4_en_2: now also J11.3 (Pin_3)
- net Multiplexer_COM: now also R25.1
- net Write_RX: now also J12.1 (Pin_1)
- net Write_TX: now also J12.2 (Pin_2)
- net at R29.1: now also SW1.1
- new net: CR1.1, Q13.1 (G), Q14.1 (G), R42.2
- new net: Q13.3 (D), Q14.3 (D)
- new net: R43.1, SW1.3
- new net 3.3v: J1.1 (Pin_1), J5.2 (Pin_2), Q13.2 (S)
- new net 3v_1: C36.1, CR1.2, CR2.2, U7.2 (OUTPUT)
Other:
- added sheet line (untitled.kicad_sch)
- moved on the sheet: J4
